File: Walking-Setup/Treadmill-Illumination/Treadmill-Illumination-v2-1206-smd/Treadmill-Illumination-v2-1206.kicad_pcb (KiCad board)
At the start: 2 copper layers, 56 x 34 mm, 11 parts, among them J2 S2B-PH-SM4-TB

Commit message: include type in filename
Parts:
- D10, D11, D14, D15: footprint LED_SMD:LED_0603_1608Metric_Pad1.05x0.95mm_HandSolder -> LED_SMD:LED_1206_3216Metric_Pad1.42x1.75mm_HandSolder
- moved D10 0.14 mm to (123.0, 96.0)
Routing:
- net Net-(D10-K): track 20.0 -> 18.7 mm
- net Net-(D14-K): track 19.9 -> 18.7 mm

Commit message: use page settings for silkscreen, ready PCBs for order
Other:
- board text added: "${COMMENT1}"
- board text added: "${REVISION} ${ISSUE_DATE}"
- board text added: "${TITLE}"
- board text removed: "Treadmill Illumination"
- board text removed: "v2.1 2026-09-28"
Changed lines of the file:
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@@
 	)
 	(paper "A4")
+	(title_block
+		(title "Treadmill Illumination 1206")
+		(date "2026-09-29")
+		(rev "v2.1")
+		(company "Reiserlab @ Janelia | HHMI")
+		(comment 1 "https://reiserlab.github.io/Fly-Lab-Gear/")
+	)
 	(layers
 		(0 "F.Cu" signal)
@@
 		(layer "Edge.Cuts")
 	)
-	(gr_text "v2.1 2026-09-28"
-		(at 109.25 121.75 0)
+	(gr_text "${COMMENT1}"
+		(at 79.62 119.04 0)
 		(layer "F.SilkS")
 		(effects
@@
 		)
 	)
+	(gr_text "${REVISION} ${ISSUE_DATE}"
+		(at 108.14 121.09 0)
+		(layer "F.SilkS")
+		(effects
+			(font
+				(size 0.8 0.8)
+				(thickness 0.1)
+			)
+			(justify left bottom)
+		)
+	)
 	(gr_text "+5V"
-		(at 121 113.5 0)
-		(layer "F.SilkS")
+		(at 120.97 113.4 0)
+		(layer "F.SilkS" knockout)
 		(effects
 			(font
@@
 	)
 	(gr_text "GND"
-		(at 127.25 113.5 0)
-		(layer "F.SilkS")
+		(at 127.27 113.4 0)
+		(layer "F.SilkS" knockout)
 		(effects
 			(font
@@
 		)
 	)
-	(gr_text "Treadmill Illumination"
-		(at 83.25 121.75 0)
+	(gr_text "${TITLE}"
+		(at 79.53 121.17 0)
 		(layer "F.SilkS")
 		(effects
 			(font
-				(size 1.5 1.5)
-				(thickness 0.3)
+				(size 1.3 1.3)
+				(thickness 0.26)
 				(bold yes)
 			)
 			(justify left bottom)
+		)
+	)
+	(gr_text "${REVISION} ${ISSUE_DATE}"
+		(at 91.13 121.15 0)
+		(layer "B.SilkS")
+		(effects
+			(font
+				(size 0.8 0.8)
+				(thickness 0.1)
+			)
+			(justify left bottom mirror)
+		)
+	)
+	(gr_text "${COMMENT1}"
+		(at 119.2 119.14 0)
+		(layer "B.SilkS")
+		(effects
+			(font
+				(size 0.8 0.8)
+				(thickness 0.1)
+			)
+			(justify left bottom mirror)
 		)
 	)
@@
 		)
 	)
-	(gr_text "v2.1 2026-09-28"
-		(at 98 121 0)
+	(gr_text "${TITLE}"
+		(at 119.5 121.06 0)
 		(layer "B.SilkS")
 		(effects
 			(font
-				(size 1 1)
-				(thickness 0.125)
-			)
-			(justify left bottom mirror)
-		)
-	)
-	(gr_text "Treadmill Illumination"
-		(at 123.5 121 0)
-		(layer "B.SilkS")
-		(effects
-			(font
-				(size 1.5 1.5)
-				(thickness 0.3)
+				(size 1.3 1.3)
+				(thickness 0.26)
 				(bold yes)
 			)
