File: Walking-Setup/Treadmill-Illumination/Treadmill-Illumination-v2-1206-smd/Treadmill-Illumination-v2-1206.kicad_sch (KiCad schematic)
At the start: 11 parts, among them J2 S2B-PH-SM4-TB

Commit message: Update schematic title block to match PCB page
Other:
- title: Treadmill Illumination -> Treadmill Illumination 1206
Changed lines of the file:
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@@
 	(paper "USLetter")
 	(title_block
-		(title "Treadmill Illumination")
-		(date "2026-09-28")
+		(title "Treadmill Illumination 1206")
+		(date "2026-09-29")
 		(rev "v2.1")
 		(company "Reiserlab @ Janelia | HHMI")
+		(comment 1 "https://reiserlab.github.io/Fly-Lab-Gear/")
 	)
 	(junction
