File: Walking-Setup/Treadmill-Illumination/Treadmill-Illumination-v2-tht/Treadmill-Illumination-v2-tht.kicad_pcb (KiCad board)
At the start: 2 copper layers, 61 x 34 mm, 11 parts, among them J2 S2B-PH-K-S-GW

Commit message: use page settings for silkscreen, ready PCBs for order
Other:
- board text added: "${REVISION} ${ISSUE_DATE}"
- board text added: "${TITLE}"
- board text added: "https://reiserlab.github.io/Fly-Lab-Gear/"
- board text removed: "Treadmill Illumination"
- board text removed: "v2.1 2026-09-28"
Changed lines of the file:
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@@
 	)
 	(paper "A4")
+	(title_block
+		(title "Treadmill Illumination THT")
+		(date "2026-09-29")
+		(rev "v2.1")
+		(company "Reiserlab @ Janelia | HHMI")
+	)
 	(layers
 		(0 "F.Cu" signal)
@@
 		(layer "Edge.Cuts")
 	)
-	(gr_text "v2.1 2026-09-28"
+	(gr_text "${REVISION} ${ISSUE_DATE}"
 		(at 109.25 121.75 0)
 		(layer "F.SilkS")
@@
 		)
 	)
+	(gr_text "https://reiserlab.github.io/Fly-Lab-Gear/"
+		(at 83.37 119.15 0)
+		(layer "F.SilkS")
+		(effects
+			(font
+				(size 1 1)
+				(thickness 0.15)
+			)
+			(justify left bottom)
+		)
+	)
 	(gr_text "+5V"
 		(at 125.5 114 0)
-		(layer "F.SilkS")
+		(layer "F.SilkS" knockout)
 		(effects
 			(font
 				(size 1 1)
-				(thickness 0.125)
+				(thickness 0.2)
+				(bold yes)
 			)
 			(justify left bottom)
@@
 	(gr_text "GND"
 		(at 129.3 114 0)
-		(layer "F.SilkS")
+		(layer "F.SilkS" knockout)
 		(effects
 			(font
 				(size 1 1)
-				(thickness 0.125)
+				(thickness 0.2)
+				(bold yes)
 			)
 			(justify left bottom)
 		)
 	)
-	(gr_text "Treadmill Illumination"
-		(at 83.25 121.75 0)
+	(gr_text "${TITLE}"
+		(at 78.74 121.7 0)
 		(layer "F.SilkS")
 		(effects
@@
 		)
 	)
-	(gr_text "v2.1 2026-09-28"
-		(at 98 121 0)
+	(gr_text "${REVISION} ${ISSUE_DATE}"
+		(at 92.98 121.73 0)
 		(layer "B.SilkS")
 		(effects
@@
 		)
 	)
-	(gr_text "Treadmill Illumination"
-		(at 123.5 121 0)
+	(gr_text "https://reiserlab.github.io/Fly-Lab-Gear/"
+		(at 123.91 119.11 0)
+		(layer "B.SilkS")
+		(effects
+			(font
+				(size 1 1)
+				(thickness 0.15)
+			)
+			(justify left bottom mirror)
+		)
+	)
+	(gr_text "${TITLE}"
+		(at 123.91 121.79 0)
 		(layer "B.SilkS")
 		(effects
